File: CentralUnit/ActuatorConn.sch (KiCad schematic (older format))
At the start: 3 parts, among them J5 Conn_01x02, Q1 Q_NMOS_GDS

Commit message: Some improvements
Parts:
- added R39: 560R, Resistors_SMD:R_0603, symbol Device:R
Connections:
- net GATE: now also R39.1; no longer Q1.1 (G)
- new net: Q1.1 (G), R39.2
Other:
- moved on the sheet: R14
Changed lines of the file:
@@
 $Descr A4 11693 8268
 encoding utf-8
-Sheet 11 16
+Sheet 2 16
 Title ""
 Date ""
@@
 Wire Wire Line
 	4800 4200 4500 4200
-Text HLabel 5150 4000 2    50   Input ~ 0
+Text HLabel 5450 4000 2    50   Input ~ 0
 GATE
 $Comp
 L Device:R R5
 U 1 1 5C033959
-P 5100 4200
+P 5450 4150
 AR Path="/5C0130E7/5C033959" Ref="R5"  Part="1"
 AR Path="/5C0162C8/5C033959" Ref="R6"  Part="1"
@@
 AR Path="/5C0169FB/5C033959" Ref="R13"  Part="1"
 AR Path="/5C0169FE/5C033959" Ref="R14"  Part="1"
-F 0 "R14" H 5170 4246 50  0000 L CNN
-F 1 "10K" V 5100 4150 50  0000 L CNN
-F 2 "Resistors_SMD:R_0603" V 5030 4200 50  0001 C CNN
-F 3 "~" H 5100 4200 50  0001 C CNN
-	1    5100 4200
+F 0 "R14" H 5520 4196 50  0000 L CNN
+F 1 "10K" V 5450 4100 50  0000 L CNN
+F 2 "Resistors_SMD:R_0603" V 5380 4150 50  0001 C CNN
+F 3 "~" H 5450 4150 50  0001 C CNN
+	1    5450 4150
 	1    0    0    -1
 $EndComp
-Wire Wire Line
-	5100 4050 5100 4000
-Wire Wire Line
-	5100 4000 5150 4000
-Connection ~ 5100 4000
 $Comp
 L power:GND #PWR?
 U 1 1 5C03463D
-P 5100 4350
+P 5450 4300
 AR Path="/5C03463D" Ref="#PWR?"  Part="1"
 AR Path="/5C0130E7/5C03463D" Ref="#PWR0127"  Part="1"
@@
 AR Path="/5C0169FB/5C03463D" Ref="#PWR0151"  Part="1"
 AR Path="/5C0169FE/5C03463D" Ref="#PWR0154"  Part="1"
-F 0 "#PWR0154" H 5100 4100 50  0001 C CNN
-F 1 "GND" H 5000 4250 50  0000 C CNN
-F 2 "" H 5100 4350 50  0001 C CNN
-F 3 "" H 5100 4350 50  0001 C CNN
-	1    5100 4350
+F 0 "#PWR0154" H 5450 4050 50  0001 C CNN
+F 1 "GND" H 5350 4200 50  0000 C CNN
+F 2 "" H 5450 4300 50  0001 C CNN
+F 3 "" H 5450 4300 50  0001 C CNN
+	1    5450 4300
 	1    0    0    -1
 $EndComp
+$Comp
+L Device:R R39
+U 1 1 5C0A7800
+P 5250 4000
+AR Path="/5C0130E7/5C0A7800" Ref="R39"  Part="1"
+AR Path="/5C0162C8/5C0A7800" Ref="R40"  Part="1"
+AR Path="/5C0163D9/5C0A7800" Ref="R41"  Part="1"
+AR Path="/5C0163DC/5C0A7800" Ref="R42"  Part="1"
+AR Path="/5C016537/5C0A7800" Ref="R43"  Part="1"
+AR Path="/5C01653A/5C0A7800" Ref="R44"  Part="1"
+AR Path="/5C01653D/5C0A7800" Ref="R45"  Part="1"
+AR Path="/5C016540/5C0A7800" Ref="R46"  Part="1"
+AR Path="/5C0169FB/5C0A7800" Ref="R47"  Part="1"
+AR Path="/5C0169FE/5C0A7800" Ref="R48"  Part="1"
+F 0 "R48" V 5350 4050 50  0000 C CNN
+F 1 "560R" V 5250 4000 50  0000 C CNN
+F 2 "Resistors_SMD:R_0603" V 5180 4000 50  0001 C CNN
+F 3 "~" H 5250 4000 50  0001 C CNN
+	1    5250 4000
+	0    1    1    0
+$EndComp
+Wire Wire Line
+	5400 4000 5450 4000
 $EndSCHEMATC
