File: CentralUnit/FloorHeatingCentral.sch (KiCad schematic (older format))
At the start: 27 parts, among them J1 Conn_01x03, J2 Conn_01x03, J25 Conn_02x05_Odd_Even, J26 Conn_01x02, J3 Conn_01x19, J4 Conn_01x06, U1 ESP32-WROOM, U10 LM1117-3.3, U7 74HC595D_118, U8 74HC595D_118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

Commit message: Some improvements
Parts:
- added H1, H2: MountingHole, parts:PCB_DINrail_holder, symbol Mechanical:MountingHole
Changed lines of the file:
@@
 Wire Wire Line
 	9350 5450 9350 5100
+$Comp
+L Mechanical:MountingHole H2
+U 1 1 5C0B012C
+P 1100 6350
+F 0 "H2" H 1200 6396 50  0000 L CNN
+F 1 "MountingHole" H 1200 6305 50  0000 L CNN
+F 2 "parts:PCB_DINrail_holder" H 1100 6350 50  0001 C CNN
+F 3 "~" H 1100 6350 50  0001 C CNN
+	1    1100 6350
+	1    0    0    -1
+$EndComp
+$Comp
+L Mechanical:MountingHole H1
+U 1 1 5C0B0591
+P 1100 6150
+F 0 "H1" H 1200 6196 50  0000 L CNN
+F 1 "MountingHole" H 1200 6105 50  0000 L CNN
+F 2 "parts:PCB_DINrail_holder" H 1100 6150 50  0001 C CNN
+F 3 "~" H 1100 6150 50  0001 C CNN
+	1    1100 6150
+	1    0    0    -1
+$EndComp
 $EndSCHEMATC

Commit message: V2 with fixed SPI bus, status LED und changed flash header
Parts:
- removed J1: Conn_01x03, Pin_Headers:Pin_Header_Straight_1x03_Pitch2.54mm, symbol Connector_Generic:Conn_01x03
- removed J3: Conn_01x19, parts:12864_LCD_128x64, symbol Connector_Generic:Conn_01x19
- added D1, D2: LED, LEDs:LED_0603, symbol Device:LED
- added J1: Conn_01x02, Pin_Headers:Pin_Header_Straight_1x02_Pitch2.54mm, symbol Connector_Generic:Conn_01x02
- added J3: Conn_01x20, parts:12864_LCD_128x64, symbol Connector_Generic:Conn_01x20
- added R49, R50: 660R, Resistors_SMD:R_0603, symbol Device:R
- C16, C17: footprint Capacitors_SMD:C_0603 -> Capacitors_SMD:C_1206
Connections:
- net +3V3: now also R1.2, J3.19 (Pin_19), J3.2 (Pin_2), R50.2
- net DISP_CS: now also J3.4 (Pin_4)
- net DISP_RST: now also J3.17 (Pin_17)
- net GND: now also D1.1 (K), D2.1 (K), J1.2 (Pin_2), J3.1 (Pin_1), J3.15 (Pin_15), J3.20 (Pin_20)
- net INP0: now also U1.8 (IO32); no longer U1.21 (SDO)
- net INP1: now also U1.9 (IO33); no longer U1.22 (SD1)
- net at C1.1, U1.3 (EN): now also R1.1, J1.1 (Pin_1); no longer R1.2
- net LED: now reaches U1.37 (IO23)
- net LED: now also R49.2
- net at RV1.2: now also J3.3 (Pin_3)
- net JTAG_TCK renamed HSPI_MOSI_IO13
- net HSPI_MOSI_IO13: now also U7.14 (DS), J3.5 (Pin_5)
- net JTAG_TDI renamed HSPI_MISO_IO12
- net JTAG_TDO renamed HSPI_CS0_IO15
- net JTAG_TMS renamed HSPI_CLK_IO14
- net HSPI_CLK_IO14: now also U7.11 (SHCP), U8.11 (SHCP), J3.6 (Pin_6)
- removed net SPI2CLK: U1.17 (SD2), U7.11 (SHCP), U8.11 (SHCP)
- net SPI2MISO: no longer names the net of U1.18 (SD3)
- net SPI2MOSI: no longer names the net of U1.20 (CLK)
- net SPI2MOSI: no longer U7.14 (DS)
- new net: D2.2 (A), R50.1
- new net: D1.2 (A), R49.1
- no-connect marks 33 -> 35
Other:
- moved on the sheet: J25, R1, R35, R36, R37, R38, RV1
