File: CentralUnit/FloorHeatingCentral.sch (KiCad schematic (older format))
At the start: 34 parts, among them J1 Conn_01x02, J2 Conn_01x03, J25 Conn_02x05_Odd_Even, J26 Conn_01x02, J3 Conn_01x20, J4 Conn_01x06, U1 ESP32-WROOM, U10 LM1117-3.3, U7 74HC595D_118, U8 74HC595D_118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

Commit message: Added possibility to PWM LCD light and updated README
Parts:
- removed R51: R, Resistors_SMD:R_0603, symbol Device:R
- added Q?: Q_PMOS_GSD, symbol Device:Q_PMOS_GSD
- added R?: Inf, symbol Device:R
- added R?: 330, symbol Device:R
Connections:
- net labels added: VDD_DL
- wire segments 114 -> 117
Other:
- moved on the sheet: J3, RV1
Changed lines of the file:
@@
 L power:GND #PWR0120
 U 1 1 5C073605
-P 9550 5450
-F 0 "#PWR0120" H 9550 5200 50  0001 C CNN
-F 1 "GND" V 9550 5200 50  0000 C CNN
-F 2 "" H 9550 5450 50  0001 C CNN
-F 3 "" H 9550 5450 50  0001 C CNN
-	1    9550 5450
+P 10300 5950
+F 0 "#PWR0120" H 10300 5700 50  0001 C CNN
+F 1 "GND" V 10300 5700 50  0000 C CNN
+F 2 "" H 10300 5950 50  0001 C CNN
+F 3 "" H 10300 5950 50  0001 C CNN
+	1    10300 5950
 	-1   0    0    1
 $EndComp
@@
 L power:+3.3V #PWR0121
 U 1 1 5C073FB3
-P 9200 4650
-F 0 "#PWR0121" H 9200 4500 50  0001 C CNN
-F 1 "+3.3V" V 9200 4900 50  0000 C CNN
-F 2 "" H 9200 4650 50  0001 C CNN
-F 3 "" H 9200 4650 50  0001 C CNN
-	1    9200 4650
+P 9950 5150
+F 0 "#PWR0121" H 9950 5000 50  0001 C CNN
+F 1 "+3.3V" V 9950 5400 50  0000 C CNN
+F 2 "" H 9950 5150 50  0001 C CNN
+F 3 "" H 9950 5150 50  0001 C CNN
+	1    9950 5150
 	0    -1   -1   0
 $EndComp
@@
 L Device:R_POT RV1
 U 1 1 5C075695
-P 9350 4650
-F 0 "RV1" V 9143 4650 50  0000 C CNN
-F 1 "R_POT" V 9234 4650 50  0000 C CNN
-F 2 "Potentiometers:Potentiometer_Trimmer_Bourns_3296W" H 9350 4650 50  0001 C CNN
-F 3 "~" H 9350 4650 50  0001 C CNN
-	1    9350 4650
-	0    1    1    0
-$EndComp
-Text Label 9250 5100 3    50   ~ 0
+P 10100 5150
+F 0 "RV1" V 9893 5150 50  0000 C CNN
+F 1 "R_POT" V 9984 5150 50  0000 C CNN
+F 2 "Potentiometers:Potentiometer_Trimmer_Bourns_3296W" H 10100 5150 50  0001 C CNN
+F 3 "~" H 10100 5150 50  0001 C CNN
+	1    10100 5150
+	0    1    1    0
+$EndComp
+Text Label 10000 5600 3    50   ~ 0
 DISP_CS
 Wire Wire Line
-	9250 5100 9250 5450
-Text Label 9150 4800 3    50   ~ 0
+	10000 5600 10000 5950
+Text Label 9900 5300 3    50   ~ 0
 HSPI_MOSI_IO13
-Text Label 9050 4800 3    50   ~ 0
+Text Label 9800 5300 3    50   ~ 0
 HSPI_CLK_IO14
-NoConn ~ 8950 5450
-NoConn ~ 8850 5450
-NoConn ~ 8750 5450
-NoConn ~ 8650 5450
-NoConn ~ 8550 5450
-NoConn ~ 8450 5450
-NoConn ~ 8350 5450
-NoConn ~ 8250 5450
+NoConn ~ 9700 5950
+NoConn ~ 9600 5950
+NoConn ~ 9500 5950
+NoConn ~ 9400 5950
+NoConn ~ 9300 5950
+NoConn ~ 9200 5950
+NoConn ~ 9100 5950
+NoConn ~ 9000 5950
 $Comp
 L power:GND #PWR0122
 U 1 1 5C08433B
-P 8150 5450
-F 0 "#PWR0122" H 8150 5200 50  0001 C CNN
-F 1 "GND" V 8150 5250 50  0000 C CNN
-F 2 "" H 8150 5450 50  0001 C CNN
-F 3 "" H 8150 5450 50  0001 C CNN
-	1    8150 5450
+P 8900 5950
+F 0 "#PWR0122" H 8900 5700 50  0001 C CNN
+F 1 "GND" V 8900 5750 50  0000 C CNN
+F 2 "" H 8900 5950 50  0001 C CNN
+F 3 "" H 8900 5950 50  0001 C CNN
+	1    8900 5950
 	-1   0    0    1
 $EndComp
-Text Label 7950 5100 3    50   ~ 0
+Text Label 8700 5600 3    50   ~ 0
 DISP_RST
 Wire Wire Line
-	7950 5450 7950 5100
-NoConn ~ 8050 5450
-$Comp
-L power:+3.3V #PWR0123
-U 1 1 5C086D45
-P 7750 5450
-F 0 "#PWR0123" H 7750 5300 50  0001 C CNN
-F 1 "+3.3V" V 7750 5700 50  0000 C CNN
-F 2 "" H 7750 5450 50  0001 C CNN
-F 3 "" H 7750 5450 50  0001 C CNN
-	1    7750 5450
-	1    0    0    -1
-$EndComp
-$Comp
-L power:GND #PWR0124
-U 1 1 5C087494
-P 7650 5450
-F 0 "#PWR0124" H 7650 5200 50  0001 C CNN
-F 1 "GND" V 7650 5200 50  0000 C CNN
-F 2 "" H 7650 5450 50  0001 C CNN
-F 3 "" H 7650 5450 50  0001 C CNN
-	1    7650 5450
-	-1   0    0    1
-$EndComp
+	8700 5950 8700 5600
+NoConn ~ 8800 5950
 $Sheet
 S 3850 4750 800  350
@@
 L power:GND #PWR0115
 U 1 1 5C10CC8D
-P 9500 4650
-F 0 "#PWR0115" H 9500 4400 50  0001 C CNN
-F 1 "GND" V 9500 4400 50  0000 C CNN
-F 2 "" H 9500 4650 50  0001 C CNN
-F 3 "" H 9500 4650 50  0001 C CNN
-	1    9500 4650
+P 10250 5150
+F 0 "#PWR0115" H 10250 4900 50  0001 C CNN
+F 1 "GND" V 10250 4900 50  0000 C CNN
+F 2 "" H 10250 5150 50  0001 C CNN
+F 3 "" H 10250 5150 50  0001 C CNN
+	1    10250 5150
 	0    -1   -1   0
 $EndComp
@@
 L power:+3.3V #PWR0215
 U 1 1 5C1102D5
-P 9450 5450
-F 0 "#PWR0215" H 9450 5300 50  0001 C CNN
-F 1 "+3.3V" V 9450 5700 50  0000 C CNN
-F 2 "" H 9450 5450 50  0001 C CNN
-F 3 "" H 9450 5450 50  0001 C CNN
-	1    9450 5450
+P 10200 5950
+F 0 "#PWR0215" H 10200 5800 50  0001 C CNN
+F 1 "+3.3V" V 10200 6200 50  0000 C CNN
+F 2 "" H 10200 5950 50  0001 C CNN
+F 3 "" H 10200 5950 50  0001 C CNN
+	1    10200 5950
 	1    0    0    -1
 $EndComp
@@
 L Connector_Generic:Conn_01x20 J3
 U 1 1 5C37801C
-P 8650 5650
-F 0 "J3" V 8775 5596 50  0000 C CNN
-F 1 "Conn_01x20" V 8866 5596 50  0000 C CNN
-F 2 "parts:12864_LCD_128x64" H 8650 5650 50  0001 C CNN
-F 3 "~" H 8650 5650 50  0001 C CNN
-	1    8650 5650
-	0    1    1    0
-$EndComp
-NoConn ~ 7850 5450
+P 9400 6150
+F 0 "J3" V 9525 6096 50  0000 C CNN
+F 1 "Conn_01x20" V 9616 6096 50  0000 C CNN
+F 2 "parts:12864_LCD_128x64" H 9400 6150 50  0001 C CNN
+F 3 "~" H 9400 6150 50  0001 C CNN
+	1    9400 6150
+	0    1    1    0
+$EndComp
+NoConn ~ 8600 5950
 Wire Wire Line
 	8150 3900 8150 4500
@@
 $EndComp
 Wire Wire Line
-	9050 4800 9050 5450
-Wire Wire Line
-	9150 4800 9150 5450
+	9800 5300 9800 5950
+Wire Wire Line
+	9900 5300 9900 5950
 Wire Wire Line
 	9600 2100 9400 2100
@@
 Text Label 9400 2400 0    50   ~ 0
 RXD
-$Comp
-L Device:R R51
-U 1 1 5D7CE8C5
-P 9700 4950
-F 0 "R51" V 9493 4950 50  0000 C CNN
-F 1 "R" V 9584 4950 50  0000 C CNN
-F 2 "Resistors_SMD:R_0603" V 9630 4950 50  0001 C CNN
-F 3 "~" H 9700 4950 50  0001 C CNN
-	1    9700 4950
-	0    1    1    0
-$EndComp
-Wire Wire Line
-	9350 4800 9350 4950
-Wire Wire Line
-	9550 4950 9350 4950
-Connection ~ 9350 4950
-Wire Wire Line
-	9350 4950 9350 5450
-Wire Wire Line
-	9850 4950 10200 4950
-Text Label 10200 4950 2    50   ~ 0
+Wire Wire Line
+	10100 5300 10100 5950
+$Comp
+L Device:Q_PMOS_GSD Q?
+U 1 1 5D8C6A7D
+P 7200 5900
+F 0 "Q?" H 7406 5854 50  0000 L CNN
+F 1 "Q_PMOS_GSD" H 7406 5945 50  0000 L CNN
+F 2 "" H 7400 6000 50  0001 C CNN
+F 3 "~" H 7200 5900 50  0001 C CNN
+	1    7200 5900
+	1    0    0    1
+$EndComp
+$Comp
+L power:GND #PWR0124
+U 1 1 5C087494
+P 8400 5950
+F 0 "#PWR0124" H 8400 5700 50  0001 C CNN
+F 1 "GND" V 8500 5950 50  0000 C CNN
+F 2 "" H 8400 5950 50  0001 C CNN
+F 3 "" H 8400 5950 50  0001 C CNN
+	1    8400 5950
+	-1   0    0    1
+$EndComp
+$Comp
+L power:+3.3V #PWR0123
+U 1 1 5C086D45
+P 7300 5600
+F 0 "#PWR0123" H 7300 5450 50  0001 C CNN
+F 1 "+3.3V" V 7300 5850 50  0000 C CNN
+F 2 "" H 7300 5600 50  0001 C CNN
+F 3 "" H 7300 5600 50  0001 C CNN
+	1    7300 5600
+	1    0    0    -1
+$EndComp
+$Comp
+L Device:R R?
+U 1 1 5D8D7CAF
+P 6650 5750
+F 0 "R?" H 6720 5796 50  0000 L CNN
+F 1 "Inf" H 6720 5705 50  0000 L CNN
+F 2 "" V 6580 5750 50  0001 C CNN
+F 3 "~" H 6650 5750 50  0001 C CNN
+	1    6650 5750
+	1    0    0    -1
+$EndComp
+Wire Wire Line
+	7300 5700 7300 5600
+Connection ~ 7300 5600
+$Comp
+L Device:R R?
+U 1 1 5D8DB005
+P 6850 5900
+F 0 "R?" H 6920 5946 50  0000 L CNN
+F 1 "330" H 6920 5855 50  0000 L CNN
+F 2 "" V 6780 5900 50  0001 C CNN
+F 3 "~" H 6850 5900 50  0001 C CNN
+	1    6850 5900
+	0    1    1    0
+$EndComp
+Wire Wire Line
+	6700 5900 6650 5900
+Wire Wire Line
+	6450 5900 6650 5900
+Wire Wire Line
+	8500 5950 8500 5600
+Text Label 6450 5900 0    50   ~ 0
 IO0
+Connection ~ 6650 5900
+Wire Wire Line
+	6650 5600 7300 5600
+Text Label 8500 5600 3    50   ~ 0
+VDD_DL
+Text Label 7300 6400 1    50   ~ 0
+VDD_DL
+Wire Wire Line
+	7300 6100 7300 6400
 $EndSCHEMATC
