File: CentralUnit/FloorHeatingCentral.kicad_pcb (KiCad board)
At the start: 2 copper layers, 110 x 110 mm, 72 parts, among them J1 Screw_Terminal_01x02, J10 Screw_Terminal_01x02, J11 Screw_Terminal_01x02, J12 Screw_Terminal_01x02, J13 Screw_Terminal_01x02, J14 Screw_Terminal_01x04, J15 Conn_01x04_Male, J16 Conn_01x04_Male, J17 Conn_01x04_Male, J18 Conn_01x04_Male, J2 Conn_02x05_Odd_Even, J3 Conn_01x20, J4 Screw_Terminal_01x02, J5 Screw_Terminal_01x02, J6 Screw_Terminal_01x02, J7 Screw_Terminal_01x02, J8 Screw_Terminal_01x02, J9 Screw_Terminal_01x02, Q1 Q_NMOS_GDS, Q10 Q_NMOS_GDS, Q11 Q_NMOS_GDS, Q2 Q_NMOS_GDS, Q3 Q_NMOS_GDS, Q4 Q_NMOS_GDS, Q5 Q_NMOS_GDS, Q6 Q_NMOS_GDS, Q7 Q_NMOS_GDS, Q8 Q_NMOS_GDS, Q9 Q_NMOS_GDS, U1 ESP32-DevKitC, U2 74HC595D_118, U3 74HC595D_118, U4 RFM69-ATSHA-breakout, U5 MP1584, U6 LM1117-5.0

Commit message: Updates
Connections:
- J3 pad 6: /VSPI_CLK -> /VSPI_SCK
- U2 pad 11: /VSPI_CLK -> /VSPI_SCK
- U3 pad 11: /VSPI_CLK -> /VSPI_SCK
Routing:
- net /VSPI_SCK: track 13.4 -> 90.3 mm, vias 0 -> 1
- net /VSPI_CLK: track 25.3 -> 0.00 mm
