File: RoomUnit/RoomUnit.sch (KiCad schematic (older format))
At the start: 43 parts, among them J1 Conn_01x03, J2 Conn_01x03, J3 Conn_01x03, J4 Conn_01x03, Q1 BC817, U1 LM1117-3.3, U2 ESP-12F, U3 ISO1540DR, U4 1.3\"_128x64OLED_I2C, U5 LTR-303ALS-01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

Commit message: Bugfixes: Wrong use of GPIO15, removed header for GPIO2
Parts:
- removed J2: Conn_01x03, Pin_Headers:Pin_Header_Straight_1x03_Pitch2.54mm, symbol Connector_Generic:Conn_01x03
Connections:
- net +3V3: now also R9.2; no longer R6.2
- net GND: now also R6.2
Other:
- moved on the sheet: J1, R6, R8, R9
Changed lines of the file:
@@
 L Device:R R8
 U 1 1 5C061166
-P 4700 2300
-F 0 "R8" V 4650 2450 50  0000 C CNN
-F 1 "10k" V 4700 2300 50  0000 C CNN
-F 2 "Resistors_SMD:R_0603" V 4630 2300 50  0001 C CNN
-F 3 "~" H 4700 2300 50  0001 C CNN
-	1    4700 2300
+P 4700 2800
+F 0 "R8" V 4650 2950 50  0000 C CNN
+F 1 "10k" V 4700 2800 50  0000 C CNN
+F 2 "Resistors_SMD:R_0603" V 4630 2800 50  0001 C CNN
+F 3 "~" H 4700 2800 50  0001 C CNN
+	1    4700 2800
 	0    1    1    0
 $EndComp
@@
 L Device:R R6
 U 1 1 5C061FE9
-P 4450 1500
-F 0 "R6" V 4400 1650 50  0000 C CNN
-F 1 "10k" V 4450 1500 50  0000 C CNN
-F 2 "Resistors_SMD:R_0603" V 4380 1500 50  0001 C CNN
-F 3 "~" H 4450 1500 50  0001 C CNN
-	1    4450 1500
-	0    1    1    0
-$EndComp
-Text Label 5150 2300 2    50   ~ 0
+P 4450 2100
+F 0 "R6" V 4400 2250 50  0000 C CNN
+F 1 "10k" V 4450 2100 50  0000 C CNN
+F 2 "Resistors_SMD:R_0603" V 4380 2100 50  0001 C CNN
+F 3 "~" H 4450 2100 50  0001 C CNN
+	1    4450 2100
+	0    1    1    0
+$EndComp
+Text Label 5150 2800 2    50   ~ 0
 GPIO0
-Text Label 5150 3000 2    50   ~ 0
+Text Label 4900 1500 2    50   ~ 0
 GPIO2
-Text Label 4900 1500 2    50   ~ 0
+Text Label 4900 2100 2    50   ~ 0
 GPIO15
 Wire Wire Line
-	4850 2300 5150 2300
-Wire Wire Line
-	4900 1500 4600 1500
+	4850 2800 5150 2800
+Wire Wire Line
+	4900 2100 4600 2100
 $Comp
 L Device:R R7
@@
 Wire Wire Line
 	4900 1700 4600 1700
-Wire Wire Line
-	4300 1700 4300 1500
 Text Label 1650 1350 0    50   ~ 0
 CH_PD
 Wire Wire Line
 	1650 1350 1950 1350
-Connection ~ 4300 1500
 $Comp
 L Connector_Generic:Conn_01x03 J1
 U 1 1 5C070E7B
-P 4350 2300
-F 0 "J1" H 4268 2617 50  0000 C CNN
-F 1 "Conn_01x03" H 4268 2526 50  0000 C CNN
-F 2 "Pin_Headers:Pin_Header_Straight_1x03_Pitch2.54mm" H 4350 2300 50  0001 C CNN
-F 3 "~" H 4350 2300 50  0001 C CNN
-	1    4350 2300
+P 4350 2800
+F 0 "J1" H 4268 3117 50  0000 C CNN
+F 1 "Conn_01x03" H 4268 3026 50  0000 C CNN
+F 2 "Pin_Headers:Pin_Header_Straight_1x03_Pitch2.54mm" H 4350 2800 50  0001 C CNN
+F 3 "~" H 4350 2800 50  0001 C CNN
+	1    4350 2800
 	-1   0    0    -1
 $EndComp
@@
 L power:+3.3V #PWR0125
 U 1 1 5C07ABA4
-P 4550 2400
-F 0 "#PWR0125" H 4550 2250 50  0001 C CNN
-F 1 "+3.3V" H 4565 2573 50  0000 C CNN
-F 2 "" H 4550 2400 50  0001 C CNN
-F 3 "" H 4550 2400 50  0001 C CNN
-	1    4550 2400
-	-1   0    0    1
-$EndComp
-$Comp
-L power:GND #PWR0126
-U 1 1 5C07B538
-P 4550 2200
-F 0 "#PWR0126" H 4550 1950 50  0001 C CNN
-F 1 "GND" H 4555 2027 50  0000 C CNN
-F 2 "" H 4550 2200 50  0001 C CNN
-F 3 "" H 4550 2200 50  0001 C CNN
-	1    4550 2200
-	-1   0    0    1
-$EndComp
-$Comp
-L Device:R R9
-U 1 1 5C07CB75
-P 4700 3000
-F 0 "R9" V 4650 3150 50  0000 C CNN
-F 1 "10k" V 4700 3000 50  0000 C CNN
-F 2 "Resistors_SMD:R_0603" V 4630 3000 50  0001 C CNN
-F 3 "~" H 4700 3000 50  0001 C CNN
-	1    4700 3000
-	0    1    1    0
-$EndComp
-Wire Wire Line
-	4850 3000 5150 3000
-$Comp
-L Connector_Generic:Conn_01x03 J2
-U 1 1 5C07CB7D
-P 4350 3000
-F 0 "J2" H 4268 3317 50  0000 C CNN
-F 1 "Conn_01x03" H 4268 3226 50  0000 C CNN
-F 2 "Pin_Headers:Pin_Header_Straight_1x03_Pitch2.54mm" H 4350 3000 50  0001 C CNN
-F 3 "~" H 4350 3000 50  0001 C CNN
-	1    4350 3000
-	-1   0    0    -1
-$EndComp
-$Comp
-L power:+3.3V #PWR0127
-U 1 1 5C07CB83
-P 4550 3100
-F 0 "#PWR0127" H 4550 2950 50  0001 C CNN
-F 1 "+3.3V" H 4565 3273 50  0000 C CNN
-F 2 "" H 4550 3100 50  0001 C CNN
-F 3 "" H 4550 3100 50  0001 C CNN
-	1    4550 3100
-	-1   0    0    1
-$EndComp
-$Comp
-L power:GND #PWR0128
-U 1 1 5C07CB89
 P 4550 2900
-F 0 "#PWR0128" H 4550 2650 50  0001 C CNN
-F 1 "GND" H 4555 2727 50  0000 C CNN
+F 0 "#PWR0125" H 4550 2750 50  0001 C CNN
+F 1 "+3.3V" H 4565 3073 50  0000 C CNN
 F 2 "" H 4550 2900 50  0001 C CNN
 F 3 "" H 4550 2900 50  0001 C CNN
 	1    4550 2900
 	-1   0    0    1
+$EndComp
+$Comp
+L power:GND #PWR0126
+U 1 1 5C07B538
+P 4550 2700
+F 0 "#PWR0126" H 4550 2450 50  0001 C CNN
+F 1 "GND" H 4555 2527 50  0000 C CNN
+F 2 "" H 4550 2700 50  0001 C CNN
+F 3 "" H 4550 2700 50  0001 C CNN
+	1    4550 2700
+	-1   0    0    1
+$EndComp
+$Comp
+L Device:R R9
+U 1 1 5C07CB75
+P 4450 1500
+F 0 "R9" V 4400 1650 50  0000 C CNN
+F 1 "10k" V 4450 1500 50  0000 C CNN
+F 2 "Resistors_SMD:R_0603" V 4380 1500 50  0001 C CNN
+F 3 "~" H 4450 1500 50  0001 C CNN
+	1    4450 1500
+	0    1    1    0
+$EndComp
+Wire Wire Line
+	4600 1500 4900 1500
+$Comp
+L power:GND #PWR0128
+U 1 1 5C07CB89
+P 4300 2100
+F 0 "#PWR0128" H 4300 1850 50  0001 C CNN
+F 1 "GND" H 4305 1927 50  0000 C CNN
+F 2 "" H 4300 2100 50  0001 C CNN
+F 3 "" H 4300 2100 50  0001 C CNN
+	1    4300 2100
+	0    1    1    0
 $EndComp
 Text Label 3650 1750 2    50   ~ 0
@@
 	4300 1200 4300 1300
 Connection ~ 4300 1300
-Wire Wire Line
-	4300 1300 4300 1500
 $Comp
 L power:GND #PWR0129
@@
 	0    1    1    0
 $EndComp
+Wire Wire Line
+	4300 1300 4300 1500
+Connection ~ 4300 1500
+Wire Wire Line
+	4300 1500 4300 1700
 $EndSCHEMATC

Commit message: Major work changing over to 868MHz solution. Current state unfinished
Parts:
- removed C10, C9: 100u, Capacitors_SMD:C_0603, symbol Device:C
- removed C6, C7: C, Capacitors_SMD:C_0603, symbol Device:C
- removed J3: Conn_01x03, parts:ScrewTerminal_3x2.54, symbol Connector_Generic:Conn_01x03
- removed R10, R11: 10k, Resistors_SMD:R_0603, symbol Device:R
- removed R3, R4: 2.7k, Resistors_SMD:R_0603, symbol Device:R
- removed U3: ISO1540DR, digikey-footprints:SOIC-8_W3.9mm, symbol dk_Digital-Isolators:ISO1540DR
- removed U6: BME680, footprints:Bosch_LGA-8_3x3mm_P0.8mm_ClockwisePinNumbering, symbol Sensor:BME680
- removed U7: BME280, Housings_LGA:Bosch_LGA-8_2.5x2.5mm_Pitch0.65mm_ClockwisePinNumbering, symbol Sensor:BME280
- added AE1: Antenna, Connector_PinHeader_2.54mm:PinHeader_1x01_P2.54mm_Horizontal, symbol Device:Antenna
- added J2: Conn_01x06_Female, Connector_PinHeader_2.54mm:PinHeader_1x06_P2.54mm_Vertical, symbol Connector:Conn_01x06_Female
- added JP1: SolderJumper_2_Bridged, Jumper:SolderJumper-2_P1.3mm_Open_RoundedPad1.0x1.5mm, symbol Jumper:SolderJumper_2_Bridged
- added U3: RFM69HW, RF_Module:HOPERF_RFM69HW, symbol RF_Module:RFM69HW
Connections:
- net +3V3: now also J2.1 (Pin_1), J2.5 (Pin_5), J2.6 (Pin_6), JP1.2 (B)
- net +5V: now also JP1.1 (A)
- net GND: now also J2.2 (Pin_2)
- net SCL: now also J2.3 (Pin_3)
- net SDA: now also J2.4 (Pin_4)
- new net: AE1.1 (A), U3.10 (ANA)
- new net: U3.11 (GND), U3.9 (GND)
Other:
- moved on the sheet: C8, U5
